File: pcb/SplitFlap.kicad_pcb (KiCad board)
At the start: 2 copper layers, 35 x 35 mm, 17 parts, among them U1 PCF8575DBR, U2 ULN2003

Commit message: Update version number
Other:
- board text added: "SplitFlap v2"
- board text removed: "SplitFlap v1"
Changed lines of the file:
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@@
 		(layer "Edge.Cuts")
 	)
-	(gr_text "SplitFlap v1"
+	(gr_text "SplitFlap v2"
 		(at 146 62 0)
 		(layer "F.SilkS")
